File: pcb/chargerDischarger.V6.brd (EAGLE design)
At the start: 185 x 116.5 mm, 83 parts, among them CON1 B6B-EH-A, CON2 SQT-110-01-F-D-RA, K101 ORWH, K102 RT424F05054

Commit message: new board versions
Connections:
- net CHAR: now also PIC1.15, R101.1; no longer PIC1.14, R103.1
- net DISC: now also PIC1.14, R103.1; no longer PIC1.15, R101.1
Routing:
- net CHAR: track 10.7 -> 6.02 mm
- net DISC: track 6.80 -> 10.7 mm
Changed lines of the file:
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@@
 <?xml version="1.0" encoding="utf-8"?>
 <!DOCTYPE eagle SYSTEM "eagle.dtd">
-<eagle version="9.4.2">
+<eagle version="9.5.1">
 <drawing>
 <settings>
@@
 <layer number="14" name="Route14" color="1" fill="6" visible="no" active="no"/>
 <layer number="15" name="Route15" color="4" fill="6" visible="no" active="no"/>
-<layer number="16" name="Bottom" color="1" fill="1" visible="no" active="yes"/>
+<layer number="16" name="Bottom" color="1" fill="1" visible="yes" active="yes"/>
 <layer number="17" name="Pads" color="2" fill="1" visible="yes" active="yes"/>
 <layer number="18" name="Vias" color="2" fill="1" visible="yes" active="yes"/>
@@
 <layer number="20" name="Dimension" color="24" fill="1" visible="yes" active="yes"/>
 <layer number="21" name="tPlace" color="7" fill="1" visible="yes" active="yes"/>
-<layer number="22" name="bPlace" color="7" fill="1" visible="no" active="yes"/>
+<layer number="22" name="bPlace" color="7" fill="1" visible="yes" active="yes"/>
 <layer number="23" name="tOrigins" color="15" fill="1" visible="yes" active="yes"/>
-<layer number="24" name="bOrigins" color="15" fill="1" visible="no" active="yes"/>
+<layer number="24" name="bOrigins" color="15" fill="1" visible="yes" active="yes"/>
 <layer number="25" name="tNames" color="7" fill="1" visible="yes" active="yes"/>
-<layer number="26" name="bNames" color="7" fill="1" visible="no" active="yes"/>
+<layer number="26" name="bNames" color="7" fill="1" visible="yes" active="yes"/>
 <layer number="27" name="tValues" color="7" fill="1" visible="no" active="yes"/>
 <layer number="28" name="bValues" color="7" fill="1" visible="no" active="yes"/>
@@
 <layer number="38" name="bTest" color="7" fill="1" visible="no" active="yes"/>
 <layer number="39" name="tKeepout" color="4" fill="11" visible="yes" active="yes"/>
-<layer number="40" name="bKeepout" color="1" fill="11" visible="no" active="yes"/>
+<layer number="40" name="bKeepout" color="1" fill="11" visible="yes" active="yes"/>
 <layer number="41" name="tRestrict" color="4" fill="10" visible="yes" active="yes"/>
-<layer number="42" name="bRestrict" color="1" fill="10" visible="no" active="yes"/>
+<layer number="42" name="bRestrict" color="1" fill="10" visible="yes" active="yes"/>
 <layer number="43" name="vRestrict" color="2" fill="10" visible="no" active="yes"/>
 <layer number="44" name="Drills" color="7" fill="1" visible="no" active="yes"/>
@@
 <layer number="50" name="dxf" color="7" fill="1" visible="no" active="no"/>
 <layer number="51" name="tDocu" color="7" fill="1" visible="yes" active="yes"/>
-<layer number="52" name="bDocu" color="7" fill="1" visible="no" active="yes"/>
+<layer number="52" name="bDocu" color="7" fill="1" visible="yes" active="yes"/>
 <layer number="53" name="tGND_GNDA" color="7" fill="9" visible="no" active="no"/>
 <layer number="54" name="bGND_GNDA" color="1" fill="9" visible="no" active="no"/>
@@
 <attribute name="NAME" x="133.4" y="61.7" size="1.27" layer="26" rot="MR180" align="center"/>
 </element>
-<element name="PR701" library="Pasives" library_urn="urn:adsk.eagle:library:2793478" package="TO-220HEATSINK" package3d_urn="urn:adsk.eagle:package:5417999/5" value="1" x="140" y="20" smashed="yes" rot="R90">
+<element name="PR701" library="Pasives" library_urn="urn:adsk.eagle:library:2793478" package="TO-220HEATSINK" package3d_urn="urn:adsk.eagle:package:5417999/7" value="1" x="140" y="20" smashed="yes" rot="R90">
 <attribute name="NAME" x="130" y="16.5" size="1.27" layer="25" font="vector" rot="R90"/>
 </element>
-<element name="PR702" library="Pasives" library_urn="urn:adsk.eagle:library:2793478" package="TO-220HEATSINK" package3d_urn="urn:adsk.eagle:package:5417999/5" value="1" x="110" y="20" smashed="yes" rot="R90">
+<element name="PR702" library="Pasives" library_urn="urn:adsk.eagle:library:2793478" package="TO-220HEATSINK" package3d_urn="urn:adsk.eagle:package:5417999/7" value="1" x="110" y="20" smashed="yes" rot="R90">
 <attribute name="NAME" x="100" y="16.5" size="1.27" layer="25" font="vector" rot="R90"/>
 </element>
-<element name="PR703" library="Pasives" library_urn="urn:adsk.eagle:library:2793478" package="TO-220HEATSINK" package3d_urn="urn:adsk.eagle:package:5417999/5" value="1" x="80" y="20" smashed="yes" rot="R90">
+<element name="PR703" library="Pasives" library_urn="urn:adsk.eagle:library:2793478" package="TO-220HEATSINK" package3d_urn="urn:adsk.eagle:package:5417999/7" value="1" x="80" y="20" smashed="yes" rot="R90">
 <attribute name="NAME" x="70" y="16.5" size="1.27" layer="25" font="vector" rot="R90"/>
 </element>
@@
 <wire x1="111.63" y1="76" x2="116" y2="71.63" width="2.5" layer="16"/>
 <wire x1="116" y1="71.63" x2="116" y2="30.65" width="2.5" layer="16"/>
-<wire x1="133.9" y1="22.54" x2="124.11" y2="22.54" width="2.5" layer="16"/>
+<wire x1="133.2" y1="22.54" x2="124.11" y2="22.54" width="2.5" layer="16"/>
 <wire x1="124.11" y1="22.54" x2="116" y2="30.65" width="2.5" layer="16"/>
-<wire x1="73.9" y1="22.54" x2="103.9" y2="22.54" width="2.5" layer="16"/>
-<wire x1="103.9" y1="22.54" x2="107.89" y2="22.54" width="2.5" layer="16"/>
+<wire x1="73.2" y1="22.54" x2="103.2" y2="22.54" width="2.5" layer="16"/>
+<wire x1="103.2" y1="22.54" x2="107.89" y2="22.54" width="2.5" layer="16"/>
 <wire x1="107.89" y1="22.54" x2="116" y2="30.65" width="2.5" layer="16"/>
 </signal>
@@
 </signal>
 <signal name="CHAR">
-<contactref element="R103" pad="1"/>
-<contactref element="PIC1" pad="14"/>
-<wire x1="64.05" y1="89.15" x2="62.06" y2="91.14" width="0.2" layer="1"/>
-<wire x1="64.05" y1="89.15" x2="71.94" y2="89.15" width="0.2" layer="1"/>
-</signal>
-<signal name="DISC">
 <contactref element="R101" pad="1"/>
 <contactref element="PIC1" pad="15"/>
-<wire x1="64.91" y1="103.6" x2="63.6" y2="103.6" width="0.2" layer="1"/>
-<wire x1="63.6" y1="103.6" x2="62.05" y2="102.05" width="0.2" layer="1"/>
-<wire x1="62.05" y1="102.05" x2="62.06" y2="102.04" width="0.2" layer="1"/>
-<wire x1="62.06" y1="102.04" x2="62.06" y2="98.76" width="0.2" layer="1"/>
+<wire x1="64.91" y1="103.6" x2="62.06" y2="100.75" width="0.2" layer="1"/>
+<wire x1="62.06" y1="100.75" x2="62.06" y2="98.76" width="0.2" layer="1"/>
+</signal>
+<signal name="DISC">
+<contactref element="R103" pad="1"/>
+<contactref element="PIC1" pad="14"/>
+<wire x1="62.06" y1="91.14" x2="63.66" y2="91.14" width="0.2" layer="1"/>
+<wire x1="63.66" y1="91.14" x2="65.65" y2="89.15" width="0.2" layer="1"/>
+<wire x1="65.65" y1="89.15" x2="71.94" y2="89.15" width="0.2" layer="1"/>
 </signal>
 <signal name="I_SENS">
