File: pcb/chargerDischarger.V6.sch (EAGLE design)
At the start: 20 parts, among them CON1 B6B-EH-A, CON2 SQT-110-01-F-D-RA

Commit message: new board versions
Connections:
- net CHAR: now also PIC1.RC4, R1.1; no longer PIC1.RC3
- net DISC: now also PIC1.RC3; no longer PIC1.RC4, R1.1
Changed lines of the file:
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@@
 <?xml version="1.0" encoding="utf-8"?>
 <!DOCTYPE eagle SYSTEM "eagle.dtd">
-<eagle version="9.4.2">
+<eagle version="9.5.1">
 <drawing>
 <settings>
@@
 </segment>
 </net>
-<net name="DISC" class="0">
+<net name="CHAR" class="0">
 <segment>
 <pinref part="R1" gate="G$1" pin="1"/>
@@
 </segment>
 </net>
-<net name="CHAR" class="0">
+<net name="DISC" class="0">
 <segment>
 <pinref part="R3" gate="G$1" pin="1"/>
@@
 <attribute name="TITLE" value="General"/>
 </part>
-<part name="PR1" library="Pasives" library_urn="urn:adsk.eagle:library:2793478" deviceset="TO-220_RESISTOR" device="" package3d_urn="urn:adsk.eagle:package:5417999/5" value="1"/>
-<part name="PR2" library="Pasives" library_urn="urn:adsk.eagle:library:2793478" deviceset="TO-220_RESISTOR" device="" package3d_urn="urn:adsk.eagle:package:5417999/5" value="1"/>
-<part name="PR3" library="Pasives" library_urn="urn:adsk.eagle:library:2793478" deviceset="TO-220_RESISTOR" device="" package3d_urn="urn:adsk.eagle:package:5417999/5" value="1"/>
+<part name="PR1" library="Pasives" library_urn="urn:adsk.eagle:library:2793478" deviceset="TO-220_RESISTOR" device="" package3d_urn="urn:adsk.eagle:package:5417999/7" value="1"/>
+<part name="PR2" library="Pasives" library_urn="urn:adsk.eagle:library:2793478" deviceset="TO-220_RESISTOR" device="" package3d_urn="urn:adsk.eagle:package:5417999/7" value="1"/>
+<part name="PR3" library="Pasives" library_urn="urn:adsk.eagle:library:2793478" deviceset="TO-220_RESISTOR" device="" package3d_urn="urn:adsk.eagle:package:5417999/7" value="1"/>
 </parts>
 <sheets>
@@
 <net name="CHAR" class="0">
 <segment>
-<label x="86.36" y="111.76" size="1.778" layer="95" xref="yes"/>
+<label x="109.22" y="114.3" size="1.778" layer="95" xref="yes"/>
+<wire x1="83.82" y1="114.3" x2="109.22" y2="114.3" width="0.1524" layer="91"/>
+<pinref part="PIC1" gate="G$1" pin="RC4"/>
+</segment>
+</net>
+<net name="DISC" class="0">
+<segment>
+<label x="87.63" y="111.76" size="1.778" layer="95" xref="yes"/>
+<wire x1="83.82" y1="111.76" x2="87.63" y2="111.76" width="0.1524" layer="91"/>
 <pinref part="PIC1" gate="G$1" pin="RC3"/>
-<wire x1="83.82" y1="111.76" x2="86.36" y2="111.76" width="0.1524" layer="91"/>
-</segment>
-</net>
-<net name="DISC" class="0">
-<segment>
-<label x="107.95" y="114.3" size="1.778" layer="95" xref="yes"/>
-<pinref part="PIC1" gate="G$1" pin="RC4"/>
-<wire x1="106.68" y1="114.3" x2="107.95" y2="114.3" width="0.1524" layer="91"/>
-<wire x1="83.82" y1="114.3" x2="106.68" y2="114.3" width="0.1524" layer="91"/>
-</segment>
-</net>
+</segment>
+</net>
